File: Board/P214-001/p214_001_001.sch (EAGLE design)
At the start: 23 parts, among them IC1 74LS07N

Commit message: new design.
Parts:
- removed SW1: (no value), special:SW_DIP-1
- added SV2: (no value), con-lstb:MA05-1
- C1: value (none) -> 104
- R4: value (none) -> 10k
- R5, R6: value (none) -> 300
Connections:
- net GND: now also R7.1, SV2.2; no longer SW1.1
- net N$17: now also SV2.5
- net N$18: now also SV2.4
- net N$25: now also PCB1.D7, R7.2
- net N$37: now also PCB1.D12, SV2.3; no longer PCB1.D7, R7.1, SW1.2
- net VCC: now also SV2.1; no longer R7.2
Other:
- moved on the sheet: R7
Changed lines of the file:
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@@
 <setting verticaltext="up"/>
 </settings>
-<grid distance="0.1" unitdist="inch" unit="inch" style="lines" multiple="1" display="no" altdistance="0.01" altunitdist="inch" altunit="inch"/>
+<grid distance="0.05" unitdist="inch" unit="inch" style="lines" multiple="1" display="no" altdistance="0.01" altunitdist="inch" altunit="inch"/>
 <layers>
 <layer number="1" name="Top" color="4" fill="1" visible="no" active="no"/>
@@
 <part name="R2" library="resistor" deviceset="R-US_" device="0204/7" value="220"/>
 <part name="R3" library="resistor" deviceset="R-US_" device="0204/7" value="220"/>
-<part name="R4" library="resistor" deviceset="R-US_" device="0204/7"/>
+<part name="R4" library="resistor" deviceset="R-US_" device="0204/7" value="10k"/>
 <part name="SUPPLY3" library="supply2" deviceset="GND" device=""/>
 <part name="SUPPLY4" library="supply2" deviceset="GND" device=""/>
@@
 <part name="REARPORT" library="con-ml" deviceset="ML10L" device=""/>
 <part name="OK1" library="optocoupler" deviceset="6N137" device="" value="TLP552"/>
-<part name="C1" library="rcl" deviceset="C-US" device="025-025X050"/>
+<part name="C1" library="rcl" deviceset="C-US" device="025-025X050" value="104"/>
 <part name="SUPPLY1" library="supply2" deviceset="VCC" device=""/>
-<part name="R5" library="resistor" deviceset="R-US_" device="0204/7"/>
+<part name="R5" library="resistor" deviceset="R-US_" device="0204/7" value="300"/>
 <part name="D1" library="diode" deviceset="1N4148" device="DO35-10"/>
 <part name="SUPPLY2" library="supply2" deviceset="GND" device=""/>
@@
 <part name="SUPPLY16" library="supply2" deviceset="VCC" device=""/>
 <part name="SUPPLY17" library="supply2" deviceset="GND" device=""/>
-<part name="R6" library="resistor" deviceset="R-US_" device="0204/7"/>
+<part name="R6" library="resistor" deviceset="R-US_" device="0204/7" value="300"/>
 <part name="LED1" library="led" deviceset="LED" device="3MM"/>
 <part name="SUPPLY18" library="supply2" deviceset="GND" device=""/>
-<part name="SW1" library="special" deviceset="SW_DIP-1" device=""/>
 <part name="R7" library="resistor" deviceset="R-US_" device="0204/7"/>
 <part name="SUPPLY19" library="supply2" deviceset="GND" device=""/>
 <part name="SUPPLY20" library="supply2" deviceset="VCC" device=""/>
+<part name="SUPPLY21" library="supply2" deviceset="GND" device=""/>
+<part name="SV2" library="con-lstb" deviceset="MA05-1" device=""/>
 </parts>
 <sheets>
@@
 <instance part="LED1" gate="G$1" x="129.54" y="15.24"/>
 <instance part="SUPPLY18" gate="GND" x="129.54" y="-7.62"/>
-<instance part="SW1" gate="G$1" x="132.08" y="71.12" rot="R270"/>
-<instance part="R7" gate="G$1" x="132.08" y="86.36" rot="R90"/>
-<instance part="SUPPLY19" gate="GND" x="132.08" y="55.88"/>
-<instance part="SUPPLY20" gate="G$1" x="132.08" y="96.52"/>
+<instance part="R7" gate="G$1" x="102.87" y="-2.54" rot="R90"/>
+<instance part="SUPPLY19" gate="GND" x="102.87" y="-10.16"/>
+<instance part="SUPPLY20" gate="G$1" x="119.38" y="96.52"/>
+<instance part="SUPPLY21" gate="GND" x="111.76" y="80.01"/>
+<instance part="SV2" gate="G$1" x="129.54" y="82.55" rot="R180"/>
 </instances>
 <busses>
@@
 <segment>
 <pinref part="SUPPLY20" gate="G$1" pin="VCC"/>
-<pinref part="R7" gate="G$1" pin="2"/>
-<wire x1="132.08" y1="93.98" x2="132.08" y2="91.44" width="0.1524" layer="91"/>
+<wire x1="119.38" y1="93.98" x2="119.38" y2="87.63" width="0.1524" layer="91"/>
+<pinref part="SV2" gate="G$1" pin="1"/>
+<wire x1="119.38" y1="87.63" x2="121.92" y2="87.63" width="0.1524" layer="91"/>
 </segment>
 </net>
@@
 </segment>
 <segment>
-<pinref part="SW1" gate="G$1" pin="1"/>
+<pinref part="R7" gate="G$1" pin="1"/>
 <pinref part="SUPPLY19" gate="GND" pin="GND"/>
-<wire x1="132.08" y1="58.42" x2="132.08" y2="63.5" width="0.1524" layer="91"/>
+</segment>
+<segment>
+<pinref part="SUPPLY21" gate="GND" pin="GND"/>
+<wire x1="121.92" y1="85.09" x2="111.76" y2="85.09" width="0.1524" layer="91"/>
+<wire x1="111.76" y1="85.09" x2="111.76" y2="82.55" width="0.1524" layer="91"/>
+<pinref part="SV2" gate="G$1" pin="2"/>
 </segment>
 </net>
@@
 <pinref part="OK1" gate="A" pin="VO"/>
 <wire x1="111.76" y1="48.26" x2="104.14" y2="48.26" width="0.1524" layer="91"/>
-<wire x1="104.14" y1="48.26" x2="104.14" y2="27.94" width="0.1524" layer="91"/>
 <pinref part="PCB1" gate="G$1" pin="RX"/>
+<wire x1="104.14" y1="35.56" x2="104.14" y2="27.94" width="0.1524" layer="91"/>
 <wire x1="104.14" y1="27.94" x2="81.28" y2="27.94" width="0.1524" layer="91"/>
+<wire x1="104.14" y1="48.26" x2="104.14" y2="35.56" width="0.1524" layer="91"/>
 </segment>
 </net>
@@
 <pinref part="PCB1" gate="G$1" pin="D2"/>
 <wire x1="81.28" y1="35.56" x2="96.52" y2="35.56" width="0.1524" layer="91"/>
-<wire x1="96.52" y1="35.56" x2="96.52" y2="86.36" width="0.1524" layer="91"/>
+<wire x1="96.52" y1="35.56" x2="96.52" y2="59.69" width="0.1524" layer="91"/>
+<wire x1="96.52" y1="59.69" x2="96.52" y2="86.36" width="0.1524" layer="91"/>
 <wire x1="96.52" y1="86.36" x2="-5.08" y2="86.36" width="0.1524" layer="91"/>
 <wire x1="-5.08" y1="86.36" x2="-5.08" y2="40.64" width="0.1524" layer="91"/>
 <pinref part="FRONTPORT" gate="1" pin="14"/>
 <wire x1="-5.08" y1="40.64" x2="5.08" y2="40.64" width="0.1524" layer="91"/>
+<wire x1="96.52" y1="59.69" x2="121.92" y2="59.69" width="0.1524" layer="91"/>
+<junction x="96.52" y="59.69"/>
+<pinref part="SV2" gate="G$1" pin="5"/>
+<wire x1="121.92" y1="77.47" x2="121.92" y2="59.69" width="0.1524" layer="91"/>
 </segment>
 </net>
@@
 <pinref part="PCB1" gate="G$1" pin="D3"/>
 <wire x1="81.28" y1="38.1" x2="93.98" y2="38.1" width="0.1524" layer="91"/>
-<wire x1="93.98" y1="38.1" x2="93.98" y2="83.82" width="0.1524" layer="91"/>
+<wire x1="93.98" y1="38.1" x2="93.98" y2="62.23" width="0.1524" layer="91"/>
+<wire x1="93.98" y1="62.23" x2="93.98" y2="83.82" width="0.1524" layer="91"/>
 <wire x1="93.98" y1="83.82" x2="35.56" y2="83.82" width="0.1524" layer="91"/>
 <wire x1="35.56" y1="83.82" x2="35.56" y2="43.18" width="0.1524" layer="91"/>
 <pinref part="FRONTPORT" gate="1" pin="15"/>
 <wire x1="35.56" y1="43.18" x2="20.32" y2="43.18" width="0.1524" layer="91"/>
+<wire x1="93.98" y1="62.23" x2="119.38" y2="62.23" width="0.1524" layer="91"/>
+<junction x="93.98" y="62.23"/>
+<wire x1="119.38" y1="62.23" x2="119.38" y2="80.01" width="0.1524" layer="91"/>
+<pinref part="SV2" gate="G$1" pin="4"/>
+<wire x1="119.38" y1="80.01" x2="121.92" y2="80.01" width="0.1524" layer="91"/>
 </segment>
 </net>
@@
 <pinref part="FRONTPORT" gate="1" pin="10"/>
 <wire x1="-12.7" y1="35.56" x2="5.08" y2="35.56" width="0.1524" layer="91"/>
+<wire x1="-12.7" y1="35.56" x2="-12.7" y2="2.54" width="0.1524" layer="91"/>
+<pinref part="PCB1" gate="G$1" pin="D7"/>
+<wire x1="81.28" y1="48.26" x2="102.87" y2="48.26" width="0.1524" layer="91"/>
+<wire x1="102.87" y1="48.26" x2="102.87" y2="2.54" width="0.1524" layer="91"/>
+<wire x1="-12.7" y1="2.54" x2="102.87" y2="2.54" width="0.1524" layer="91"/>
+<pinref part="R7" gate="G$1" pin="2"/>
+<junction x="102.87" y="2.54"/>
 </segment>
 </net>
@@
 <net name="N$37" class="0">
 <segment>
-<pinref part="R7" gate="G$1" pin="1"/>
-<pinref part="SW1" gate="G$1" pin="2"/>
-<wire x1="132.08" y1="81.28" x2="132.08" y2="80.01" width="0.1524" layer="91"/>
-<pinref part="PCB1" gate="G$1" pin="D7"/>
-<wire x1="132.08" y1="80.01" x2="132.08" y2="78.74" width="0.1524" layer="91"/>
-<wire x1="81.28" y1="48.26" x2="102.87" y2="48.26" width="0.1524" layer="91"/>
-<wire x1="102.87" y1="48.26" x2="102.87" y2="80.01" width="0.1524" layer="91"/>
-<wire x1="102.87" y1="80.01" x2="132.08" y2="80.01" width="0.1524" layer="91"/>
-<junction x="132.08" y="80.01"/>
-</segment>
-</net>
+<pinref part="PCB1" gate="G$1" pin="D12"/>
+<wire x1="81.28" y1="60.96" x2="81.28" y2="71.12" width="0.1524" layer="91"/>
+<pinref part="SV2" gate="G$1" pin="3"/>
+<wire x1="121.92" y1="82.55" x2="115.57" y2="82.55" width="0.1524" layer="91"/>
+<wire x1="115.57" y1="82.55" x2="115.57" y2="71.12" width="0.1524" layer="91"/>
+<wire x1="115.57" y1="71.12" x2="81.28" y2="71.12" width="0.1524" layer="91"/>
+</segment>
+</net>

Commit message: i2c socket
Parts:
- added C2: (no value), rcl:C-US050-075X075
Connections:
- net GND: now also C2.2
- net VCC: now also C2.1
Changed lines of the file:
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@@
 <setting verticaltext="up"/>
 </settings>
-<grid distance="0.05" unitdist="inch" unit="inch" style="lines" multiple="1" display="no" altdistance="0.01" altunitdist="inch" altunit="inch"/>
+<grid distance="0.1" unitdist="inch" unit="inch" style="lines" multiple="1" display="no" altdistance="0.01" altunitdist="inch" altunit="inch"/>
 <layers>
 <layer number="1" name="Top" color="4" fill="1" visible="no" active="no"/>
@@
 <part name="SUPPLY21" library="supply2" deviceset="GND" device=""/>
 <part name="SV2" library="con-lstb" deviceset="MA05-1" device=""/>
+<part name="C2" library="rcl" deviceset="C-US" device="050-075X075"/>
 </parts>
 <sheets>
@@
 <instance part="SUPPLY21" gate="GND" x="111.76" y="80.01"/>
 <instance part="SV2" gate="G$1" x="129.54" y="82.55" rot="R180"/>
+<instance part="C2" gate="G$1" x="172.72" y="91.44"/>
 </instances>
 <busses>
@@
 <pinref part="C1" gate="G$1" pin="1"/>
 <junction x="165.1" y="93.98"/>
+<pinref part="C2" gate="G$1" pin="1"/>
+<wire x1="165.1" y1="93.98" x2="172.72" y2="93.98" width="0.1524" layer="91"/>
 </segment>
 <segment>
@@
 <pinref part="C1" gate="G$1" pin="2"/>
 <junction x="165.1" y="86.36"/>
-</segment>
-<segment>
+<pinref part="C2" gate="G$1" pin="2"/>
+<wire x1="172.72" y1="86.36" x2="165.1" y2="86.36" width="0.1524" layer="91"/>
+</segment>
+<segment>

Commit message: new design.
Parts:
- removed <USB>D+, <USB>D-, <USB>GND, <USB>VBUS: (no value), wirepad:1,6/0,9
- added SV3: USB, con-lstb:MA04-1
- R7: value (none) -> 10k
- SV1: value (none) -> Analog
- SV2: value (none) -> RTC
Connections:
- removed net N$25: <USB>VBUS.P, FRONTPORT.10, PCB1.D7, R7.2
- new net N$39: FRONTPORT.10, SV3.2
- net GND: now also FRONTPORT.8, SV3.4; no longer <USB>GND.P, FRONTPORT.7
- net N$14: now also FRONTPORT.14; no longer FRONTPORT.11
- net N$15: now also FRONTPORT.15; no longer FRONTPORT.12
- net N$16: now also FRONTPORT.16; no longer FRONTPORT.13
- net N$17: now also FRONTPORT.12; no longer FRONTPORT.14
- net N$18: now also FRONTPORT.13; no longer FRONTPORT.15
- net N$22: now also SV3.3; no longer <USB>D-.P
- net N$24: now also FRONTPORT.11, PCB1.D7, R7.2, SV3.1; no longer <USB>D+.P, FRONTPORT.8
- net VCC: now also FRONTPORT.7; no longer FRONTPORT.16
Other:
- moved on the sheet: C1, C2, D1, FRONTPORT, GND, IC1A, LED1, OK1, R1, R2, R3, R4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
