File: Board/P214-001/p214_001_001.brd (EAGLE design)
At the start: 70.8 x 71.1 mm, 23 parts, among them IC1 74LS07N

Commit message: new design.
Parts:
- removed SW1: (no value), special:EDG-01
- added SV2: (no value), con-lstb:MA05-1
- C1: value (none) -> 104
- R4: value (none) -> 10k
- R5, R6: value (none) -> 300
- moved R5 48.6 mm to (26.7, 45.7), turned to 0 degrees
- moved R7 45.3 mm to (15.2, 59.7), turned to 90 degrees
- moved VCC 20.4 mm to (5.08, 2.54)
- moved GND 12.8 mm to (7.62, 2.54)
- moved R1 8.52 mm to (21.6, 15.2), turned to 0 degrees
- moved R2 6.84 mm to (8.89, 12.7), turned to 0 degrees
- moved IC1 6.48 mm to (8.89, 27.9)
- moved OK1 5.68 mm to (41.9, 8.89)
- moved C1 5.39 mm to (52.1, 12.7), turned to 0 degrees
- moved REARPORT 5.24 mm to (25.4, 11.4)
- moved FRONTPORT 5.08 mm to (38.1, 59.7)
- moved PCB1 5.08 mm to (16.5, 19.1)
- moved R4 4.58 mm to (62.2, 11.4)
- moved R3 2.84 mm to (59.7, 11.4)
- moved D1 2.84 mm to (57.1, 10.2)
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Connections:
- net GND: now also R7.1, SV2.2; no longer SW1.1
- net N$17: now also SV2.5
- net N$18: now also SV2.4
- net N$25: now also PCB1.D7, R7.2
- net N$37: now also PCB1.D12, SV2.3; no longer PCB1.D7, R7.1, SW1.2
- net VCC: now also SV2.1; no longer R7.2
Routing:
- net N$30: track 0.00 -> 78.7 mm, vias 0 -> 2
- net N$34: track 0.00 -> 77.3 mm, vias 0 -> 4
- net N$21: track 0.00 -> 67.8 mm, vias 0 -> 4
- net N$33: track 0.00 -> 67.8 mm, vias 0 -> 2
- net N$32: track 0.00 -> 65.3 mm, vias 0 -> 4
- net N$31: track 0.00 -> 65.3 mm, vias 0 -> 2
- net VCC: track 168.3 -> 211.9 mm, vias 4 -> 11
- net N$20: track 68.6 -> 26.5 mm, vias 2 -> 0
- net N$18: track 15.2 -> 57.1 mm, vias 2 -> 3
- net N$17: track 29.7 -> 67.8 mm, vias 3 -> 4
- net N$19: track 56.9 -> 33.0 mm
- net N$25: track 30.5 -> 54.4 mm
- net GND: track 232.5 -> 254.1 mm, vias 4 -> 15
- net N$7: track 67.1 -> 48.0 mm, vias 2 -> 0
- net N$5: track 20.3 -> 2.54 mm
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Other:
- board text removed: "Analog"
- board text removed: "GND"
- board text removed: "USB"
- board text removed: "Vcc"

Commit message: i2c socket
Parts:
- added C2: (no value), rcl:C050-075X075
Connections:
- net GND: now also C2.2
- net VCC: now also C2.1
Routing:
- net GND: track 254.1 -> 273.1 mm, vias 15 -> 16
- net VCC: track 211.9 -> 218.7 mm, vias 11 -> 13
- net N$19: track 33.0 -> 27.9 mm
- net N$6: track 56.4 -> 59.7 mm
- net N$29: track 37.4 -> 39.2 mm
- net N$15: track 62.8 -> 62.0 mm
- net N$33: track 67.8 -> 67.1 mm
Changed lines of the file:
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@@
 <attribute name="OC_FARNELL" value="unknown" x="63.5" y="53.34" size="1.778" layer="27" rot="R90" display="off"/>
 </element>
+<element name="C2" library="rcl" package="C050-075X075" value="" x="11.43" y="7.62" rot="R270"/>
 </elements>
 <signals>
@@
 <wire x1="53.34" y1="12.7" x2="53.34" y2="5.08" width="0.4064" layer="16"/>
 <via x="30.48" y="10.16" extent="1-16" drill="0.6"/>
-<wire x1="7.62" y1="2.54" x2="7.62" y2="7.62" width="0.4064" layer="16"/>
+<wire x1="7.62" y1="2.54" x2="7.62" y2="5.08" width="0.4064" layer="16"/>
+<wire x1="7.62" y1="5.08" x2="7.62" y2="7.62" width="0.4064" layer="16"/>
 <wire x1="7.62" y1="7.62" x2="7.62" y2="38.1" width="0.4064" layer="16"/>
 <wire x1="7.62" y1="38.1" x2="5.08" y2="38.1" width="0.4064" layer="16"/>
@@
 <via x="7.62" y="7.62" extent="1-16" drill="0.6"/>
 <wire x1="30.48" y1="7.62" x2="7.62" y2="7.62" width="0.4064" layer="1"/>
-<via x="55.88" y="55.88" extent="1-16" drill="0.6"/>
-<wire x1="55.88" y1="55.88" x2="46.99" y2="55.88" width="0.4064" layer="1"/>
-<wire x1="55.88" y1="55.88" x2="55.88" y2="50.8" width="0.4064" layer="16"/>
+<contactref element="SV2" pad="2"/>
+<wire x1="46.99" y1="55.88" x2="46.99" y2="43.18" width="0.4064" layer="16"/>
+<via x="46.99" y="43.18" extent="1-16" drill="0.6"/>
+<wire x1="46.99" y1="43.18" x2="55.88" y2="43.18" width="0.4064" layer="1"/>
+<via x="55.88" y="43.18" extent="1-16" drill="0.6"/>
+<wire x1="55.88" y1="43.18" x2="55.88" y2="50.8" width="0.4064" layer="16"/>
+<wire x1="63.5" y1="50.8" x2="60.96" y2="50.8" width="0.4064" layer="16"/>
 <via x="55.88" y="50.8" extent="1-16" drill="0.6"/>
 <via x="60.96" y="50.8" extent="1-16" drill="0.6"/>
 <wire x1="55.88" y1="50.8" x2="60.96" y2="50.8" width="0.4064" layer="1"/>
-<contactref element="SV2" pad="2"/>
-<wire x1="63.5" y1="50.8" x2="60.96" y2="50.8" width="0.4064" layer="16"/>
+<contactref element="C2" pad="2"/>
+<wire x1="11.43" y1="5.08" x2="7.62" y2="5.08" width="0.4064" layer="16"/>
 </signal>
 <signal name="VCC">
@@
 <wire x1="5.08" y1="20.32" x2="5.08" y2="16.51" width="0.4064" layer="16"/>
 <wire x1="5.08" y1="16.51" x2="5.08" y2="12.7" width="0.4064" layer="16"/>
-<wire x1="5.08" y1="12.7" x2="5.08" y2="2.54" width="0.4064" layer="16"/>
+<wire x1="5.08" y1="12.7" x2="5.08" y2="10.16" width="0" layer="19" extent="1-16"/>
+<wire x1="5.08" y1="12.7" x2="5.08" y2="10.16" width="0.4064" layer="16"/>
+<wire x1="5.08" y1="10.16" x2="5.08" y2="2.54" width="0.4064" layer="16"/>
 <wire x1="62.23" y1="7.62" x2="62.23" y2="10.16" width="0.4064" layer="16"/>
 <wire x1="62.23" y1="10.16" x2="54.61" y2="10.16" width="0.4064" layer="16"/>
@@
 <via x="5.08" y="16.51" extent="1-16" drill="0.6"/>
 <via x="48.26" y="16.51" extent="1-16" drill="0.6"/>
-<wire x1="5.08" y1="16.51" x2="10.16" y2="16.51" width="0.4064" layer="1"/>
+<wire x1="5.08" y1="16.51" x2="11.43" y2="16.51" width="0.4064" layer="1"/>
 <contactref element="SV2" pad="1"/>
-<wire x1="10.16" y1="16.51" x2="48.26" y2="16.51" width="0.4064" layer="1"/>
+<wire x1="11.43" y1="16.51" x2="48.26" y2="16.51" width="0.4064" layer="1"/>
 <wire x1="43.18" y1="58.42" x2="43.18" y2="48.26" width="0.4064" layer="16"/>
 <via x="43.18" y="48.26" extent="1-16" drill="0.6"/>
@@
 <via x="63.5" y="24.13" extent="1-16" drill="0.6"/>
 <wire x1="48.26" y1="24.13" x2="63.5" y2="24.13" width="0.4064" layer="1"/>
-<wire x1="10.16" y1="41.91" x2="10.16" y2="16.51" width="0.4064" layer="16"/>
-<via x="10.16" y="16.51" extent="1-16" drill="0.6"/>
+<wire x1="10.16" y1="41.91" x2="10.16" y2="17.78" width="0.4064" layer="16"/>
+<wire x1="10.16" y1="17.78" x2="11.43" y2="16.51" width="0.4064" layer="16"/>
+<via x="11.43" y="16.51" extent="1-16" drill="0.6"/>
+<contactref element="C2" pad="1"/>
+<via x="5.08" y="10.16" extent="1-16" drill="0.6"/>
+<wire x1="5.08" y1="10.16" x2="8.89" y2="10.16" width="0.4064" layer="1"/>
+<via x="8.89" y="10.16" extent="1-16" drill="0.6"/>
+<wire x1="8.89" y1="10.16" x2="11.43" y2="10.16" width="0.4064" layer="16"/>
 </signal>
 <signal name="N$1">
@@
 <contactref element="REARPORT" pad="4"/>
 <contactref element="R2" pad="2"/>
-<wire x1="12.7" y1="12.7" x2="12.7" y2="5.08" width="0.4064" layer="16"/>
+<wire x1="12.7" y1="12.7" x2="15.24" y2="12.7" width="0.4064" layer="16"/>
+<wire x1="15.24" y1="12.7" x2="15.24" y2="5.08" width="0.4064" layer="16"/>
 <wire x1="27.94" y1="10.16" x2="27.94" y2="5.08" width="0.4064" layer="16"/>
-<via x="12.7" y="5.08" extent="1-16" drill="0.6"/>
+<via x="15.24" y="5.08" extent="1-16" drill="0.6"/>
 <via x="27.94" y="5.08" extent="1-16" drill="0.6"/>
-<wire x1="12.7" y1="5.08" x2="27.94" y2="5.08" width="0.4064" layer="1"/>
+<wire x1="15.24" y1="5.08" x2="27.94" y2="5.08" width="0.4064" layer="1"/>
 </signal>
 <signal name="N$5">
@@
 <contactref element="REARPORT" pad="9"/>
 <contactref element="R3" pad="2"/>
-<wire x1="20.32" y1="12.7" x2="19.05" y2="11.43" width="0.4064" layer="16"/>
-<wire x1="19.05" y1="11.43" x2="19.05" y2="3.81" width="0.4064" layer="16"/>
-<wire x1="19.05" y1="3.81" x2="19.05" y2="2.54" width="0.4064" layer="16"/>
-<wire x1="19.05" y1="2.54" x2="58.42" y2="2.54" width="0.4064" layer="16"/>
-<wire x1="58.42" y1="2.54" x2="59.69" y2="2.54" width="0.4064" layer="16"/>
-<wire x1="59.69" y1="2.54" x2="59.69" y2="3.81" width="0.4064" layer="16"/>
-<wire x1="59.69" y1="3.81" x2="59.69" y2="7.62" width="0.4064" layer="16"/>
+<wire x1="20.32" y1="12.7" x2="17.78" y2="12.7" width="0.4064" layer="16"/>
+<wire x1="17.78" y1="12.7" x2="17.78" y2="2.54" width="0.4064" layer="16"/>
+<wire x1="17.78" y1="2.54" x2="59.69" y2="2.54" width="0.4064" layer="16"/>
+<wire x1="59.69" y1="2.54" x2="59.69" y2="7.62" width="0.4064" layer="16"/>
 </signal>
 <signal name="N$7">
@@
 <contactref element="PCB1" pad="MISO]"/>
 <wire x1="35.56" y1="60.96" x2="36.83" y2="59.69" width="0.4064" layer="16"/>
-<wire x1="36.83" y1="59.69" x2="36.83" y2="46.99" width="0.4064" layer="16"/>
-<via x="36.83" y="46.99" extent="1-16" drill="0.6"/>
-<wire x1="36.83" y1="46.99" x2="58.42" y2="46.99" width="0.4064" layer="1"/>
+<wire x1="36.83" y1="59.69" x2="36.83" y2="48.26" width="0.4064" layer="16"/>
+<via x="36.83" y="48.26" extent="1-16" drill="0.6"/>
+<wire x1="36.83" y1="48.26" x2="38.1" y2="46.99" width="0.4064" layer="1"/>
+<wire x1="38.1" y1="46.99" x2="58.42" y2="46.99" width="0.4064" layer="1"/>
 <via x="58.42" y="46.99" extent="1-16" drill="0.6"/>
 <wire x1="58.42" y1="46.99" x2="58.42" y2="20.32" width="0.4064" layer="16"/>
@@
 <contactref element="FRONTPORT" pad="19"/>
 <contactref element="R5" pad="2"/>
-<wire x1="45.72" y1="58.42" x2="45.72" y2="43.18" width="0.4064" layer="16"/>
-<wire x1="30.48" y1="45.72" x2="33.02" y2="45.72" width="0.4064" layer="16"/>
-<wire x1="33.02" y1="45.72" x2="33.02" y2="43.18" width="0.4064" layer="16"/>
-<via x="33.02" y="43.18" extent="1-16" drill="0.6"/>
-<via x="45.72" y="43.18" extent="1-16" drill="0.6"/>
-<wire x1="45.72" y1="43.18" x2="33.02" y2="43.18" width="0.4064" layer="1"/>
+<wire x1="45.72" y1="58.42" x2="45.72" y2="50.8" width="0.4064" layer="16"/>
+<wire x1="30.48" y1="45.72" x2="30.48" y2="50.8" width="0.4064" layer="16"/>
+<via x="30.48" y="50.8" extent="1-16" drill="0.6"/>
+<via x="45.72" y="50.8" extent="1-16" drill="0.6"/>
+<wire x1="45.72" y1="50.8" x2="30.48" y2="50.8" width="0.4064" layer="1"/>
 </signal>
 <signal name="N$11">
@@
 <contactref element="FRONTPORT" pad="24"/>
 <wire x1="40.64" y1="35.56" x2="40.64" y2="41.91" width="0.4064" layer="16"/>
-<wire x1="40.64" y1="41.91" x2="52.07" y2="41.91" width="0.4064" layer="1"/>
-<via x="52.07" y="41.91" extent="1-16" drill="0.6"/>
+<wire x1="40.64" y1="41.91" x2="53.34" y2="41.91" width="0.4064" layer="1"/>
+<via x="53.34" y="41.91" extent="1-16" drill="0.6"/>
 <via x="40.64" y="41.91" extent="1-16" drill="0.6"/>
 <wire x1="50.8" y1="60.96" x2="52.07" y2="59.69" width="0.4064" layer="16"/>
-<wire x1="52.07" y1="41.91" x2="52.07" y2="59.69" width="0.4064" layer="16"/>
+<wire x1="53.34" y1="41.91" x2="52.07" y2="43.18" width="0.4064" layer="16"/>
+<wire x1="52.07" y1="43.18" x2="52.07" y2="59.69" width="0.4064" layer="16"/>
 </signal>
 <signal name="N$21">
@@
 <wire x1="10.16" y1="58.42" x2="10.16" y2="44.45" width="0.4064" layer="16"/>
 <via x="10.16" y="44.45" extent="1-16" drill="0.6"/>
-<wire x1="10.16" y1="44.45" x2="36.83" y2="44.45" width="0.4064" layer="1"/>
-<via x="36.83" y="44.45" extent="1-16" drill="0.6"/>
-<wire x1="36.83" y1="44.45" x2="36.83" y2="21.59" width="0.4064" layer="16"/>
+<wire x1="10.16" y1="44.45" x2="35.56" y2="44.45" width="0.4064" layer="1"/>
+<wire x1="35.56" y1="44.45" x2="36.83" y2="43.18" width="0.4064" layer="1"/>
+<via x="36.83" y="43.18" extent="1-16" drill="0.6"/>
+<wire x1="36.83" y1="43.18" x2="36.83" y2="21.59" width="0.4064" layer="16"/>
 <wire x1="36.83" y1="21.59" x2="38.1" y2="20.32" width="0.4064" layer="16"/>
 </signal>
@@
 <wire x1="63.5" y1="53.34" x2="60.96" y2="53.34" width="0.4064" layer="16"/>
 <via x="60.96" y="53.34" extent="1-16" drill="0.6"/>
-<wire x1="60.96" y1="53.34" x2="54.61" y2="53.34" width="0.4064" layer="1"/>
+<wire x1="60.96" y1="53.34" x2="55.88" y2="53.34" width="0.4064" layer="1"/>
 <wire x1="20.32" y1="35.56" x2="20.32" y2="49.53" width="0.4064" layer="16"/>
 <via x="20.32" y="49.53" extent="1-16" drill="0.6"/>
-<wire x1="20.32" y1="49.53" x2="54.61" y2="49.53" width="0.4064" layer="1"/>
-<via x="54.61" y="49.53" extent="1-16" drill="0.6"/>
-<wire x1="54.61" y1="49.53" x2="54.61" y2="53.34" width="0.4064" layer="16"/>
-<via x="54.61" y="53.34" extent="1-16" drill="0.6"/>
+<wire x1="20.32" y1="49.53" x2="53.34" y2="49.53" width="0.4064" layer="1"/>
+<via x="53.34" y="49.53" extent="1-16" drill="0.6"/>
+<wire x1="53.34" y1="49.53" x2="53.34" y2="53.34" width="0.4064" layer="16"/>
+<wire x1="53.34" y1="53.34" x2="55.88" y2="53.34" width="0.4064" layer="16"/>
+<via x="55.88" y="53.34" extent="1-16" drill="0.6"/>
 </signal>
 </signals>

Commit message: new design.
Parts:
- removed <USB>D+, <USB>D-, <USB>GND, <USB>VBUS: (no value), wirepad:1,6/0,9
- added SV3: USB, con-lstb:MA04-1
- R7: value (none) -> 10k
- SV1: value (none) -> Analog
- SV2: value (none) -> RTC
- moved R5 18.5 mm to (8.89, 40.6)
- moved R6 17.8 mm to (8.89, 43.2)
- moved R7 15.3 mm to (8.89, 45.7), turned to 0 degrees
- moved R1 12.7 mm to (8.89, 15.2)
- moved SV2 5.08 mm to (63.5, 48.3)
- moved SV1 2.54 mm to (6.35, 53.3)
- moved D1 1.27 mm to (58.4, 10.2)
- moved R3 1.27 mm to (61.0, 11.4)
- moved R4 1.27 mm to (63.5, 11.4)
- moved C2 1.27 mm to (10.2, 7.62)
Connections:
- removed net N$25: <USB>VBUS.1, FRONTPORT.10, PCB1.D7, R7.2
- new net N$39: FRONTPORT.10, SV3.2
- net GND: now also FRONTPORT.8, SV3.4; no longer <USB>GND.1, FRONTPORT.7
- net N$14: now also FRONTPORT.14; no longer FRONTPORT.11
- net N$15: now also FRONTPORT.15; no longer FRONTPORT.12
- net N$16: now also FRONTPORT.16; no longer FRONTPORT.13
- net N$17: now also FRONTPORT.12; no longer FRONTPORT.14
- net N$18: now also FRONTPORT.13; no longer FRONTPORT.15
- net N$22: now also SV3.3; no longer <USB>D-.1
- net N$24: now also FRONTPORT.11, PCB1.D7, R7.2, SV3.1; no longer <USB>D+.1, FRONTPORT.8
- net VCC: now also FRONTPORT.7; no longer FRONTPORT.16
Routing:
- net N$25: track 54.4 -> 0.00 mm, vias 2 -> 0
- net N$24: track 30.5 -> 69.6 mm, vias 2 -> 4
- net N$39: track 0.00 -> 29.7 mm, vias 0 -> 2
- net N$19: track 27.9 -> 50.8 mm
- net N$22: track 55.1 -> 34.8 mm
- net N$35: track 7.62 -> 25.4 mm, vias 0 -> 2
- net N$11: track 60.2 -> 46.8 mm, vias 4 -> 2
- net N$17: track 67.8 -> 80.5 mm, vias 4 -> 3
- net N$5: track 2.54 -> 15.2 mm, vias 0 -> 2
- net N$6: track 59.7 -> 47.5 mm, vias 0 -> 2
- net VCC: track 218.7 -> 207.0 mm, vias 13 -> 11
- net N$14: track 48.3 -> 59.5 mm
- net N$2: track 12.7 -> 22.9 mm, vias 0 -> 2
- net N$20: track 26.5 -> 35.6 mm, vias 0 -> 2
- net N$8: track 34.8 -> 43.2 mm, vias 0 -> 2
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Other:
- board size 70.8 x 71.1 mm -> 71.1 x 71.1 mm

Commit message: new design.
Routing:
- net N$18: track 51.1 -> 53.3 mm, vias 4 -> 5
- net N$37: track 57.7 -> 55.9 mm
- net N$14: track 59.5 -> 57.7 mm
- net N$17: track 80.5 -> 81.3 mm
Changed lines of the file:
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@@
 <wire x1="38.1" y1="60.96" x2="38.1" y2="66.04" width="0.4064" layer="16"/>
 <via x="38.1" y="66.04" extent="1-16" drill="0.6"/>
-<wire x1="38.1" y1="66.04" x2="60.96" y2="66.04" width="0.4064" layer="1"/>
-<via x="60.96" y="66.04" extent="1-16" drill="0.6"/>
-<wire x1="60.96" y1="66.04" x2="59.69" y2="64.77" width="0.4064" layer="16"/>
-<wire x1="59.69" y1="64.77" x2="59.69" y2="36.83" width="0.4064" layer="16"/>
+<wire x1="38.1" y1="66.04" x2="59.69" y2="66.04" width="0.4064" layer="1"/>
+<via x="59.69" y="66.04" extent="1-16" drill="0.6"/>
+<wire x1="59.69" y1="66.04" x2="59.69" y2="36.83" width="0.4064" layer="16"/>
 <wire x1="59.69" y1="36.83" x2="60.96" y2="35.56" width="0.4064" layer="16"/>
 </signal>
@@
 <wire x1="40.64" y1="60.96" x2="40.64" y2="64.77" width="0.4064" layer="16"/>
 <via x="40.64" y="64.77" extent="1-16" drill="0.6"/>
-<wire x1="40.64" y1="64.77" x2="58.42" y2="64.77" width="0.4064" layer="1"/>
-<via x="58.42" y="64.77" extent="1-16" drill="0.6"/>
-<wire x1="58.42" y1="64.77" x2="58.42" y2="38.1" width="0.4064" layer="16"/>
-<via x="58.42" y="38.1" extent="1-16" drill="0.6"/>
+<wire x1="40.64" y1="64.77" x2="55.88" y2="64.77" width="0.4064" layer="1"/>
+<via x="55.88" y="64.77" extent="1-16" drill="0.6"/>
+<wire x1="55.88" y1="64.77" x2="55.88" y2="38.1" width="0.4064" layer="16"/>
+<via x="55.88" y="38.1" extent="1-16" drill="0.6"/>
 <via x="62.23" y="38.1" extent="1-16" drill="0.6"/>
-<wire x1="58.42" y1="38.1" x2="62.23" y2="38.1" width="0.4064" layer="1"/>
+<wire x1="55.88" y1="38.1" x2="62.23" y2="38.1" width="0.4064" layer="1"/>
 </signal>
 <signal name="N$17">
@@
 <wire x1="46.99" y1="67.31" x2="63.5" y2="67.31" width="0.4064" layer="1"/>
 <wire x1="63.5" y1="67.31" x2="63.5" y2="53.34" width="0.4064" layer="16"/>
-<wire x1="45.72" y1="35.56" x2="46.99" y2="36.83" width="0.4064" layer="16"/>
+<wire x1="45.72" y1="35.56" x2="45.72" y2="38.1" width="0.4064" layer="16"/>
 <via x="46.99" y="67.31" extent="1-16" drill="0.6"/>
-<wire x1="46.99" y1="36.83" x2="46.99" y2="67.31" width="0.4064" layer="16"/>
+<wire x1="45.72" y1="38.1" x2="46.99" y2="38.1" width="0.4064" layer="16"/>
+<wire x1="46.99" y1="38.1" x2="46.99" y2="39.37" width="0.4064" layer="16"/>
+<wire x1="46.99" y1="39.37" x2="46.99" y2="67.31" width="0.4064" layer="16"/>
 </signal>
 <signal name="N$18">
@@
 <contactref element="SV2" pad="4"/>
 <contactref element="FRONTPORT" pad="13"/>
-<wire x1="38.1" y1="58.42" x2="38.1" y2="55.88" width="0.4064" layer="16"/>
-<via x="41.91" y="55.88" extent="1-16" drill="0.6"/>
+<wire x1="38.1" y1="58.42" x2="38.1" y2="45.72" width="0.4064" layer="16"/>
+<wire x1="43.18" y1="35.56" x2="43.18" y2="45.72" width="0.4064" layer="16"/>
 <wire x1="63.5" y1="50.8" x2="60.96" y2="50.8" width="0.4064" layer="16"/>
-<wire x1="60.96" y1="50.8" x2="60.96" y2="53.34" width="0.4064" layer="16"/>
-<via x="60.96" y="53.34" extent="1-16" drill="0.6"/>
-<wire x1="41.91" y1="55.88" x2="41.91" y2="53.34" width="0.4064" layer="16"/>
-<wire x1="41.91" y1="53.34" x2="41.91" y2="38.1" width="0.4064" layer="16"/>
-<wire x1="41.91" y1="38.1" x2="43.18" y2="35.56" width="0.4064" layer="16"/>
-<via x="38.1" y="55.88" extent="1-16" drill="0.6"/>
-<wire x1="38.1" y1="55.88" x2="41.91" y2="55.88" width="0.4064" layer="1"/>
-<via x="41.91" y="53.34" extent="1-16" drill="0.6"/>
-<wire x1="60.96" y1="53.34" x2="41.91" y2="53.34" width="0.4064" layer="1"/>
+<via x="38.1" y="45.72" extent="1-16" drill="0.6"/>
+<via x="43.18" y="45.72" extent="1-16" drill="0.6"/>
+<via x="60.96" y="50.8" extent="1-16" drill="0.6"/>
+<wire x1="38.1" y1="45.72" x2="43.18" y2="45.72" width="0.4064" layer="1"/>
+<wire x1="60.96" y1="50.8" x2="58.42" y2="50.8" width="0.4064" layer="1"/>
+<via x="58.42" y="50.8" extent="1-16" drill="0.6"/>
+<wire x1="58.42" y1="50.8" x2="58.42" y2="45.72" width="0.4064" layer="16"/>
+<via x="58.42" y="45.72" extent="1-16" drill="0.6"/>
+<wire x1="58.42" y1="45.72" x2="43.18" y2="45.72" width="0.4064" layer="1"/>
 </signal>
 <signal name="N$20">
@@
 <contactref element="PCB1" pad="A1"/>
 <wire x1="25.4" y1="60.96" x2="24.13" y2="59.69" width="0.4064" layer="16"/>
-<wire x1="24.13" y1="59.69" x2="24.13" y2="48.26" width="0.4064" layer="16"/>
-<via x="24.13" y="48.26" extent="1-16" drill="0.6"/>
-<wire x1="24.13" y1="48.26" x2="29.21" y2="48.26" width="0.4064" layer="1"/>
-<via x="29.21" y="48.26" extent="1-16" drill="0.6"/>
-<wire x1="29.21" y1="48.26" x2="29.21" y2="21.59" width="0.4064" layer="16"/>
+<wire x1="24.13" y1="59.69" x2="24.13" y2="49.53" width="0.4064" layer="16"/>
+<via x="24.13" y="49.53" extent="1-16" drill="0.6"/>
+<wire x1="24.13" y1="49.53" x2="29.21" y2="49.53" width="0.4064" layer="1"/>
+<via x="29.21" y="49.53" extent="1-16" drill="0.6"/>
+<wire x1="29.21" y1="49.53" x2="29.21" y2="21.59" width="0.4064" layer="16"/>
 <wire x1="29.21" y1="21.59" x2="30.48" y2="20.32" width="0.4064" layer="16"/>
 </signal>
@@
 <wire x1="7.62" y1="63.5" x2="13.97" y2="63.5" width="0.4064" layer="16"/>
 <via x="13.97" y="63.5" extent="1-16" drill="0.6"/>
-<wire x1="13.97" y1="63.5" x2="13.97" y2="58.42" width="0.4064" layer="1"/>
-<wire x1="13.97" y1="58.42" x2="16.51" y2="58.42" width="0.4064" layer="1"/>
-<via x="16.51" y="58.42" extent="1-16" drill="0.6"/>
-<wire x1="16.51" y1="58.42" x2="16.51" y2="46.99" width="0.4064" layer="16"/>
+<wire x1="13.97" y1="63.5" x2="13.97" y2="57.15" width="0.4064" layer="1"/>
+<wire x1="13.97" y1="57.15" x2="16.51" y2="57.15" width="0.4064" layer="1"/>
+<via x="16.51" y="57.15" extent="1-16" drill="0.6"/>
+<wire x1="16.51" y1="57.15" x2="16.51" y2="48.26" width="0.4064" layer="16"/>
 <wire x1="5.08" y1="43.18" x2="8.89" y2="43.18" width="0.4064" layer="16"/>
 <via x="8.89" y="43.18" extent="1-16" drill="0.6"/>
-<via x="16.51" y="46.99" extent="1-16" drill="0.6"/>
-<wire x1="8.89" y1="43.18" x2="8.89" y2="46.99" width="0.4064" layer="1"/>
-<wire x1="8.89" y1="46.99" x2="16.51" y2="46.99" width="0.4064" layer="1"/>
+<via x="16.51" y="48.26" extent="1-16" drill="0.6"/>
+<wire x1="8.89" y1="43.18" x2="8.89" y2="48.26" width="0.4064" layer="1"/>
+<wire x1="8.89" y1="48.26" x2="16.51" y2="48.26" width="0.4064" layer="1"/>
 </signal>
 <signal name="N$38">
@@
 <wire x1="63.5" y1="48.26" x2="60.96" y2="48.26" width="0.4064" layer="16"/>
 <via x="60.96" y="48.26" extent="1-16" drill="0.6"/>
-<wire x1="60.96" y1="48.26" x2="59.69" y2="49.53" width="0.4064" layer="1"/>
-<wire x1="59.69" y1="49.53" x2="20.32" y2="49.53" width="0.4064" layer="1"/>
-<via x="20.32" y="49.53" extent="1-16" drill="0.6"/>
-<wire x1="20.32" y1="49.53" x2="20.32" y2="35.56" width="0.4064" layer="16"/>
+<wire x1="60.96" y1="48.26" x2="20.32" y2="48.26" width="0.4064" layer="1"/>
+<via x="20.32" y="48.26" extent="1-16" drill="0.6"/>
+<wire x1="20.32" y1="48.26" x2="20.32" y2="35.56" width="0.4064" layer="16"/>
 </signal>
 <signal name="N$39">
@@
 <wire x1="33.02" y1="60.96" x2="33.02" y2="63.5" width="0.4064" layer="16"/>
 <wire x1="10.16" y1="68.58" x2="10.16" y2="64.77" width="0.4064" layer="16"/>
-<wire x1="10.16" y1="64.77" x2="12.7" y2="64.77" width="0.4064" layer="16"/>
-<via x="12.7" y="64.77" extent="1-16" drill="0.6"/>
+<via x="10.16" y="64.77" extent="1-16" drill="0.6"/>
 <via x="33.02" y="63.5" extent="1-16" drill="0.6"/>
-<wire x1="12.7" y1="64.77" x2="31.75" y2="64.77" width="0.4064" layer="1"/>
+<wire x1="10.16" y1="64.77" x2="31.75" y2="64.77" width="0.4064" layer="1"/>
 <wire x1="31.75" y1="64.77" x2="33.02" y2="63.5" width="0.4064" layer="1"/>
 </signal>
