File: Board/P214-001/p214_001_001.brd (EAGLE design)
At the start: 71.1 x 71.1 mm, 21 parts, among them IC1 74LS07N

Commit message: new board design.
Routing:
- net VCC: track 207.0 -> 218.4 mm
- net N$21: track 73.7 -> 67.8 mm, vias 4 -> 2
- net N$9: track 42.4 -> 47.5 mm, vias 2 -> 4
- net N$30: track 72.2 -> 74.0 mm
- net N$20: track 35.6 -> 34.8 mm
- net N$17: track 81.3 -> 80.5 mm
- added copper zone on layer 1, net N$25
Changed lines of the file:
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@@
 <board>
 <plain>
-<dimension x1="0" y1="0" x2="71.12" y2="0" x3="35.56" y3="-2.54" textsize="1.778" layer="1"/>
-<dimension x1="0" y1="0" x2="0" y2="71.12" x3="-2.54" y3="35.56" textsize="1.778" layer="1"/>
 <text x="69.85" y="1.27" size="1.778" layer="1" rot="R90">P214 Rev.001 Pineapple.cc</text>
 <wire x1="0" y1="0" x2="71.12" y2="0" width="0.4064" layer="20"/>
@@
 <wire x1="71.12" y1="71.12" x2="0" y2="71.12" width="0.4064" layer="20"/>
 <wire x1="0" y1="71.12" x2="0" y2="0" width="0.4064" layer="20"/>
+<dimension x1="0" y1="0" x2="0" y2="71.12" x3="-2.54" y3="35.56" textsize="1.778" layer="20"/>
+<dimension x1="0" y1="0" x2="71.12" y2="0" x3="35.56" y3="-5.08" textsize="1.778" layer="20"/>
 </plain>
 <attributes>
@@
 <via x="52.07" y="43.18" extent="1-16" drill="0.6"/>
 <wire x1="52.07" y1="43.18" x2="60.96" y2="43.18" width="0.4064" layer="1"/>
-<wire x1="52.07" y1="43.18" x2="52.07" y2="24.13" width="0.4064" layer="16"/>
 <wire x1="48.26" y1="20.32" x2="48.26" y2="24.13" width="0.4064" layer="16"/>
-<via x="52.07" y="24.13" extent="1-16" drill="0.6"/>
+<via x="63.5" y="40.64" extent="1-16" drill="0.6"/>
 <via x="48.26" y="24.13" extent="1-16" drill="0.6"/>
-<wire x1="48.26" y1="24.13" x2="52.07" y2="24.13" width="0.4064" layer="1"/>
+<wire x1="48.26" y1="24.13" x2="63.5" y2="24.13" width="0.4064" layer="1"/>
+<wire x1="63.5" y1="24.13" x2="63.5" y2="40.64" width="0.4064" layer="1"/>
+<wire x1="63.5" y1="40.64" x2="63.5" y2="43.18" width="0.4064" layer="16"/>
 </signal>
 <signal name="N$1">
@@
 <contactref element="FRONTPORT" pad="3"/>
 <contactref element="PCB1" pad="A0"/>
-<wire x1="25.4" y1="58.42" x2="25.4" y2="38.1" width="0.4064" layer="16"/>
-<wire x1="25.4" y1="38.1" x2="24.13" y2="36.83" width="0.4064" layer="16"/>
-<wire x1="24.13" y1="36.83" x2="24.13" y2="26.67" width="0.4064" layer="16"/>
-<wire x1="27.94" y1="20.32" x2="27.94" y2="26.67" width="0.4064" layer="16"/>
-<via x="24.13" y="26.67" extent="1-16" drill="0.6"/>
-<via x="27.94" y="26.67" extent="1-16" drill="0.6"/>
-<wire x1="24.13" y1="26.67" x2="27.94" y2="26.67" width="0.4064" layer="1"/>
+<wire x1="27.94" y1="20.32" x2="26.67" y2="21.59" width="0.4064" layer="16"/>
+<wire x1="26.67" y1="21.59" x2="26.67" y2="33.02" width="0.4064" layer="16"/>
+<wire x1="25.4" y1="58.42" x2="25.4" y2="41.91" width="0.4064" layer="16"/>
+<via x="25.4" y="41.91" extent="1-16" drill="0.6"/>
+<via x="26.67" y="33.02" extent="1-16" drill="0.6"/>
+<wire x1="25.4" y1="41.91" x2="21.59" y2="41.91" width="0.4064" layer="1"/>
+<wire x1="26.67" y1="33.02" x2="21.59" y2="33.02" width="0.4064" layer="1"/>
+<via x="21.59" y="41.91" extent="1-16" drill="0.6"/>
+<via x="21.59" y="33.02" extent="1-16" drill="0.6"/>
+<wire x1="21.59" y1="41.91" x2="21.59" y2="33.02" width="0.4064" layer="16"/>
 </signal>
 <signal name="N$13">
@@
 <wire x1="46.99" y1="67.31" x2="63.5" y2="67.31" width="0.4064" layer="1"/>
 <wire x1="63.5" y1="67.31" x2="63.5" y2="53.34" width="0.4064" layer="16"/>
-<wire x1="45.72" y1="35.56" x2="45.72" y2="38.1" width="0.4064" layer="16"/>
+<wire x1="45.72" y1="35.56" x2="46.99" y2="36.83" width="0.4064" layer="16"/>
 <via x="46.99" y="67.31" extent="1-16" drill="0.6"/>
-<wire x1="45.72" y1="38.1" x2="46.99" y2="38.1" width="0.4064" layer="16"/>
-<wire x1="46.99" y1="38.1" x2="46.99" y2="39.37" width="0.4064" layer="16"/>
-<wire x1="46.99" y1="39.37" x2="46.99" y2="67.31" width="0.4064" layer="16"/>
+<wire x1="46.99" y1="36.83" x2="46.99" y2="67.31" width="0.4064" layer="16"/>
 </signal>
 <signal name="N$18">
@@
 <wire x1="5.08" y1="40.64" x2="7.62" y2="40.64" width="0.4064" layer="16"/>
 <wire x1="7.62" y1="40.64" x2="7.62" y2="24.13" width="0.4064" layer="16"/>
-<wire x1="20.32" y1="20.32" x2="20.32" y2="24.13" width="0.4064" layer="16"/>
+<wire x1="20.32" y1="20.32" x2="19.05" y2="21.59" width="0.4064" layer="16"/>
+<wire x1="19.05" y1="21.59" x2="19.05" y2="24.13" width="0.4064" layer="16"/>
 <via x="7.62" y="24.13" extent="1-16" drill="0.6"/>
-<via x="20.32" y="24.13" extent="1-16" drill="0.6"/>
-<wire x1="7.62" y1="24.13" x2="20.32" y2="24.13" width="0.4064" layer="1"/>
+<via x="19.05" y="24.13" extent="1-16" drill="0.6"/>
+<wire x1="7.62" y1="24.13" x2="19.05" y2="24.13" width="0.4064" layer="1"/>
 </signal>
 <signal name="N$23">
@@
 <contactref element="PCB1" pad="D5"/>
 <contactref element="FRONTPORT" pad="23"/>
-<wire x1="38.1" y1="35.56" x2="38.1" y2="38.1" width="0.4064" layer="16"/>
-<via x="38.1" y="38.1" extent="1-16" drill="0.6"/>
-<wire x1="38.1" y1="38.1" x2="50.8" y2="38.1" width="0.4064" layer="1"/>
-<via x="50.8" y="38.1" extent="1-16" drill="0.6"/>
-<wire x1="50.8" y1="38.1" x2="50.8" y2="58.42" width="0.4064" layer="16"/>
+<wire x1="38.1" y1="35.56" x2="38.1" y2="41.91" width="0.4064" layer="16"/>
+<via x="38.1" y="41.91" extent="1-16" drill="0.6"/>
+<wire x1="38.1" y1="41.91" x2="50.8" y2="41.91" width="0.4064" layer="1"/>
+<via x="50.8" y="41.91" extent="1-16" drill="0.6"/>
+<wire x1="50.8" y1="41.91" x2="50.8" y2="58.42" width="0.4064" layer="16"/>
 </signal>
 <signal name="N$29">
@@
 <wire x1="53.34" y1="58.42" x2="53.34" y2="39.37" width="0.4064" layer="16"/>
 <via x="53.34" y="39.37" extent="1-16" drill="0.6"/>
-<wire x1="53.34" y1="39.37" x2="21.59" y2="39.37" width="0.4064" layer="1"/>
-<via x="21.59" y="39.37" extent="1-16" drill="0.6"/>
-<wire x1="21.59" y1="39.37" x2="21.59" y2="30.48" width="0.4064" layer="16"/>
-<via x="21.59" y="30.48" extent="1-16" drill="0.6"/>
-<wire x1="21.59" y1="30.48" x2="25.4" y2="30.48" width="0.4064" layer="1"/>
-<via x="25.4" y="30.48" extent="1-16" drill="0.6"/>
-<wire x1="25.4" y1="30.48" x2="25.4" y2="20.32" width="0.4064" layer="16"/>
+<wire x1="53.34" y1="39.37" x2="24.13" y2="39.37" width="0.4064" layer="1"/>
+<via x="24.13" y="39.37" extent="1-16" drill="0.6"/>
+<wire x1="24.13" y1="39.37" x2="24.13" y2="34.29" width="0.4064" layer="16"/>
+<wire x1="24.13" y1="34.29" x2="24.13" y2="21.59" width="0.4064" layer="16"/>
+<wire x1="24.13" y1="21.59" x2="25.4" y2="20.32" width="0.4064" layer="16"/>
 </signal>
 <signal name="N$30">
@@
 <via x="45.72" y="30.48" extent="1-16" drill="0.6"/>
 <wire x1="45.72" y1="30.48" x2="45.72" y2="24.13" width="0.4064" layer="16"/>
-<wire x1="22.86" y1="20.32" x2="22.86" y2="24.13" width="0.4064" layer="16"/>
-<via x="22.86" y="24.13" extent="1-16" drill="0.6"/>
+<wire x1="22.86" y1="20.32" x2="21.59" y2="21.59" width="0.4064" layer="16"/>
+<wire x1="21.59" y1="21.59" x2="21.59" y2="24.13" width="0.4064" layer="16"/>
+<via x="21.59" y="24.13" extent="1-16" drill="0.6"/>
 <via x="45.72" y="24.13" extent="1-16" drill="0.6"/>
-<wire x1="22.86" y1="24.13" x2="45.72" y2="24.13" width="0.4064" layer="1"/>
+<wire x1="21.59" y1="24.13" x2="45.72" y2="24.13" width="0.4064" layer="1"/>
 </signal>
 <signal name="N$31">
@@
 <via x="15.24" y="59.69" extent="1-16" drill="0.6"/>
 <wire x1="33.02" y1="35.56" x2="33.02" y2="45.72" width="0.4064" layer="16"/>
-<wire x1="33.02" y1="45.72" x2="33.02" y2="55.88" width="0.4064" layer="16"/>
-<wire x1="33.02" y1="55.88" x2="35.56" y2="58.42" width="0.4064" layer="16"/>
+<wire x1="33.02" y1="45.72" x2="33.02" y2="52.07" width="0.4064" layer="16"/>
+<wire x1="33.02" y1="52.07" x2="34.29" y2="53.34" width="0.4064" layer="16"/>
+<wire x1="34.29" y1="53.34" x2="34.29" y2="57.15" width="0.4064" layer="16"/>
+<wire x1="34.29" y1="57.15" x2="35.56" y2="58.42" width="0.4064" layer="16"/>
 <wire x1="12.7" y1="45.72" x2="15.24" y2="45.72" width="0.4064" layer="16"/>
 <via x="15.24" y="45.72" extent="1-16" drill="0.6"/>
@@
 <wire x1="15.24" y1="59.69" x2="15.24" y2="45.72" width="0.4064" layer="16"/>
 </signal>
+<signal name="N$25">
+<polygon width="0.4064" layer="1">
+<vertex x="1.27" y="1.27"/>
+<vertex x="69.85" y="1.27"/>
+<vertex x="69.85" y="69.85"/>
+<vertex x="1.27" y="69.85"/>
+</polygon>
+</signal>
 </signals>
